Commit message: [Update] fully functional sim. No ros-control

File: src/robot_description/urdf/gen3_macro.xacro (robot description, xacro)
@@ -3,4 +3,262 @@
   <!-- Propagate last link name information because it is the gripper's parent link -->
   <xacro:property name="last_arm_link" value="end_effector_link"/>
+  <xacro:macro name="load_arm" params="parent:='' dof vision prefix *origin">
+  <link name="world" />
+  <joint name="world_to_base_link=" type="fixed">
+     <parent link="world"/>
+     <child link="base_link"/>
+  </joint>
+    <link name="${prefix}base_link">
+      <inertial>
+        <origin xyz="-0.000648 -0.000166 0.084487" rpy="0 0 0" />
+        <mass value="1.697" />
+        <inertia ixx="0.004622" ixy="9E-06" ixz="6E-05" iyy="0.004495" iyz="9E-06" izz="0.002079" />
+      </inertial>
+      <visual>
+        <origin xyz="0 0 0" rpy="0 0 0" />
+        <geometry>
+          <mesh filename="file://$(find robot_description)/meshes/base_link.STL" />
+        </geometry>
+        <material name="">
+          <color rgba="0.75294 0.75294 0.75294 1" />
+        </material>
+      </visual>
+      <collision>
+        <origin xyz="0 0 0" rpy="0 0 0" />
+        <geometry>
+          <mesh filename="file://$(find robot_description)/meshes/base_link.STL" />
+        </geometry>
+      </collision>
+    </link>
+    <link name="${prefix}shoulder_link">
+      <inertial>
+        <origin xyz="-2.3E-05 -0.010364 -0.07336" rpy="0 0 0" />
+        <mass value="1.377" />
+        <inertia ixx="0.00457" ixy="1E-06" ixz="2E-06" iyy="0.004831" iyz="0.000448" izz="0.001409" />
+      </inertial>
+      <visual>
+        <origin xyz="0 0 0" rpy="0 0 0" />
+        <geometry>
+          <mesh filename="file://$(find robot_description)/meshes/shoulder_link.STL" />
+        </geometry>
+        <material name="">
+          <color rgba="0.75294 0.75294 0.75294 1" />
+        </material>
+      </visual>
+      <collision>
+        <origin xyz="0 0 0" rpy="0 0 0" />
+        <geometry>
+          <mesh filename="file://$(find robot_description)/meshes/shoulder_link.STL" />
+        </geometry>
+      </collision>
+    </link>
+    <joint name="${prefix}joint_1" type="continuous">
+      <origin xyz="0 0 0.15643" rpy="-3.1416 0.0 0.0" />
+      <parent link="${prefix}base_link" />
+      <child link="${prefix}shoulder_link" />
+      <axis xyz="0 0 1" />
+      <limit effort="39" velocity="1.3963" />
+    </joint>
+    <link name="${prefix}bicep_link">
+      <inertial>
+        <origin xyz="3.5E-05 -0.208207 -0.01889" rpy="0 0 0" />
+        <mass value="1.262" />
+        <inertia ixx="0.046752" ixy="-9E-06" ixz="0" iyy="0.00085" iyz="-9.8E-05" izz="0.047188" />
+      </inertial>
+      <visual>
+        <origin xyz="0 0 0" rpy="0 0 0" />
+        <geometry>
+          <mesh filename="file://$(find robot_description)/meshes/bicep_link.STL" />
+        </geometry>
+        <material name="">
+          <color rgba="0.75294 0.75294 0.75294 1" />
+        </material>
+      </visual>
+      <collision>
+        <origin xyz="0 0 0" rpy="0 0 0" />
+        <geometry>
+          <mesh filename="file://$(find robot_description)/meshes/bicep_link.STL" />
+        </geometry>
+      </collision>
+    </link>
+    <joint name="${prefix}joint_2" type="revolute">
+      <origin xyz="0 0.005375 -0.12838" rpy="1.5708 0.0 0.0" />
+      <parent link="${prefix}shoulder_link" />
+      <child link="${prefix}bicep_link" />
+      <axis xyz="0 0 1" />
+      <limit lower="-2.24" upper="2.24" effort="39" velocity="1.3963" />
+    </joint>
+    <link name="${prefix}forearm_link">
+      <inertial>
+        <origin xyz="1.8E-05 0.076168 -0.01397" rpy="0 0 0" />
+        <mass value="0.93" />
+        <inertia ixx="0.008292" ixy="-1E-06" ixz="0" iyy="0.000628" iyz="0.000432" izz="0.008464" />
+      </inertial>
+      <visual>
+        <origin xyz="0 0 0" rpy="0 0 0" />
+        <geometry>
+          <mesh filename="file://$(find robot_description)/meshes/forearm_link.STL" />
+        </geometry>
+        <material name="">
+          <color rgba="0.75294 0.75294 0.75294 1" />
+        </material>
+      </visual>
+      <collision>
+        <origin xyz="0 0 0" rpy="0 0 0" />
+        <geometry>
+          <mesh filename="file://$(find robot_description)/meshes/forearm_link.STL" />
+        </geometry>
+      </collision>
+    </link>
+    <joint name="${prefix}joint_3" type="revolute">
+      <origin xyz="0 -0.41 0" rpy="3.1416 0 0" />
+      <parent link="${prefix}bicep_link" />
+      <child link="${prefix}forearm_link" />
+      <axis xyz="0 0 1" />
+      <limit lower="-2.57" upper="2.57" effort="39" velocity="1.3963" />
+    </joint>
+    <link name="${prefix}spherical_wrist_1_link">
+      <inertial>
+        <origin xyz="-1E-06 0.008486 -0.062937" rpy="0 0 0" />
+        <mass value="0.6781" />
+        <inertia ixx="0.001645" ixy="0" ixz="0" iyy="0.001666" iyz="-0.000234" izz="0.000389" />
+      </inertial>
+      <visual>
+        <origin xyz="0 0 0" rpy="0 0 0" />
+        <geometry>
+          <mesh filename="file://$(find robot_description)/meshes/spherical_wrist_1_link.STL" />
+        </geometry>
+        <material name="">
+          <color rgba="0.75294 0.75294 0.75294 1" />
+        </material>
+      </visual>
+      <collision>
+        <origin xyz="0 0 0" rpy="0 0 0" />
+        <geometry>
+          <mesh filename="file://$(find robot_description)/meshes/spherical_wrist_1_link.STL" />
+        </geometry>
+      </collision>
+    </link>
+    <joint name="${prefix}joint_4" type="continuous">
+      <origin xyz="0 0.20843 -0.006375" rpy="1.5708 0.0 0.0" />
+      <parent link="${prefix}forearm_link" />
+      <child link="${prefix}spherical_wrist_1_link" />
+      <axis xyz="0 0 1" />
+      <limit effort="9" velocity="1.2218" />
+    </joint>
+    <link name="${prefix}spherical_wrist_2_link">
+      <inertial>
+        <origin xyz="-1E-06 0.046429 -0.008704" rpy="0 0 0" />
+        <mass value="0.678" />
+        <inertia ixx="0.001685" ixy="0" ixz="0" iyy="0.0004" iyz="0.000255" izz="0.001696" />
+      </inertial>
+      <visual>
+        <origin xyz="0 0 0" rpy="0 0 0" />
+        <geometry>
+          <mesh filename="file://$(find robot_description)/meshes/spherical_wrist_2_link.STL" />
+        </geometry>
+        <material name="">
+          <color rgba="0.75294 0.75294 0.75294 1" />
+        </material>
+      </visual>
+      <collision>
+        <origin xyz="0 0 0" rpy="0 0 0" />
+        <geometry>
+          <mesh filename="file://$(find robot_description)/meshes/spherical_wrist_2_link.STL" />
+        </geometry>
+      </collision>
+    </link>
+    <joint name="${prefix}joint_5" type="revolute">
+      <origin xyz="0 -0.00017505 -0.10593" rpy="-1.5708 0.0 0.0" />
+      <parent link="${prefix}spherical_wrist_1_link" />
+      <child link="${prefix}spherical_wrist_2_link" />
+      <axis xyz="0 0 1" />
+      <limit lower="-2.09" upper="2.09" effort="9" velocity="1.2218" />
+    </joint>
+    <xacro:if value="${vision}">
+    <link name="${prefix}bracelet_link">
+      <inertial>
+        <origin xyz="0.000281 0.011402 -0.029798" rpy="0 0 0" />
+        <mass value="0.5" />
+        <inertia ixx="0.000587" ixy="3E-06" ixz="3E-06" iyy="0.000369" iyz="-0.000118" izz="0.000609" />
+      </inertial>
+      <visual>
+        <origin xyz="0 0 0" rpy="0 0 0" />
+        <geometry>
+          <mesh filename="file://$(find robot_description)/meshes/bracelet_with_vision_link.STL" />
+        </geometry>
+        <material name="">
+          <color rgba="0.75294 0.75294 0.75294 1" />
+        </material>
+      </visual>
+      <collision>
+        <origin xyz="0 0 0" rpy="0 0 0" />
+        <geometry>
+          <mesh filename="file://$(find robot_description)/meshes/bracelet_with_vision_link.STL" />
+        </geometry>
+      </collision>
+    </link>
+    </xacro:if>
+    <xacro:unless value="${vision}">
+    <link name="${prefix}bracelet_link">
+      <inertial>
+        <origin xyz="-9.3E-05 0.000132 -0.022905" rpy="0 0 0" />
+        <mass value="0.364" />
+        <inertia ixx="0.000214" ixy="0" ixz="1E-06" iyy="0.000223" iyz="-2E-06" izz="0.00024" />
+      </inertial>
+      <visual>
+        <origin xyz="0 0 0" rpy="0 0 0" />
+        <geometry>
+          <mesh filename="file://$(find robot_description)/meshes/bracelet_no_vision_link.STL" />
+        </geometry>
+        <material name="">
+          <color rgba="0.75294 0.75294 0.75294 1" />
+        </material>
+      </visual>
+      <collision>
+        <origin xyz="0 0 0" rpy="0 0 0" />
+        <geometry>
+          <mesh filename="file://$(find robot_description)f/meshes/bracelet_no_vision_link.STL" />
+        </geometry>
+      </collision>
+    </link>
+    </xacro:unless>
+    <joint name="${prefix}joint_6" type="continuous">
+      <origin xyz="0 0.10593 -0.00017505" rpy="1.5708 0.0 0.0" />
+      <parent link="${prefix}spherical_wrist_2_link" />
+      <child link="${prefix}bracelet_link" />
+      <axis xyz="0 0 1" />
+      <limit effort="9" velocity="1.2218" />
+    </joint>
+    <link name="${prefix}end_effector_link" />
+    <joint
+      name="${prefix}end_effector"
+      type="fixed">
+      <origin xyz="0 0 -0.0615250000000001" rpy="3.14159265358979 1.09937075168372E-32 3.14159265358979" />
+      <parent
+        link="${prefix}bracelet_link" />
+      <child
+        link="${prefix}end_effector_link" />
+      <axis
+        xyz="0 0 0" />
+    </joint>
+      <link name="${prefix}camera_link" />
+      <joint name="${prefix}camera_module" type="fixed">
+        <origin xyz="0.2 0.05639 -0.00305" rpy="3.14159265358979 3.14159265358979 0" />
+        <parent link="${prefix}end_effector_link" />
+        <child  link="${prefix}camera_link" />
+      </joint>
+      <link name="${prefix}camera_depth_frame" />
+      <joint name="${prefix}depth_module" type="fixed">
+        <origin xyz="0.0275 0.066 -0.00305" rpy="3.14159265358979 3.14159265358979 0" />
+        <parent link="${prefix}end_effector_link" />
+        <child  link="${prefix}camera_depth_frame" />
+      </joint>
+      <link name="${prefix}camera_color_frame" />
+      <joint name="${prefix}color_module" type="fixed">
+        <origin xyz="0 0.05639 -0.00305" rpy="3.14159265358979 3.14159265358979 0" />
+        <parent link="${prefix}end_effector_link" />
+        <child  link="${prefix}camera_color_frame" />
+      </joint>
    <gazebo reference="${prefix}camera_link">
     <sensor type="depth" name="intel_camera">
@@ -21,5 +279,5 @@
           </clip>
       </camera>
-      <plugin name="camera_controller" filename="libgazebo_ros_openni_kinect.so">
+      <plugin name="camera_controller" filename="libgazebo_ros_camera.so">
           <baseline>0.2</baseline>
           <alwaysOn>true</alwaysOn>
@@ -46,259 +304,4 @@
     </sensor>
   </gazebo>
-  <xacro:macro name="load_arm" params="parent:='' dof vision prefix *origin">
-    <link name="${prefix}base_link">
-      <inertial>
-        <origin xyz="-0.000648 -0.000166 0.084487" rpy="0 0 0" />
-        <mass value="1.697" />
-        <inertia ixx="0.004622" ixy="9E-06" ixz="6E-05" iyy="0.004495" iyz="9E-06" izz="0.002079" />
-      </inertial>
-      <visual>
-        <origin xyz="0 0 0" rpy="0 0 0" />
-        <geometry>
-          <mesh filename="file://$(find robot_description)/meshes/base_link.STL" />
-        </geometry>
-        <material name="">
-          <color rgba="0.75294 0.75294 0.75294 1" />
-        </material>
-      </visual>
-      <collision>
-        <origin xyz="0 0 0" rpy="0 0 0" />
-        <geometry>
-          <mesh filename="file://$(find robot_description)/meshes/base_link.STL" />
-        </geometry>
-      </collision>
-    </link>
-    <link name="${prefix}shoulder_link">
-      <inertial>
-        <origin xyz="-2.3E-05 -0.010364 -0.07336" rpy="0 0 0" />
-        <mass value="1.377" />
-        <inertia ixx="0.00457" ixy="1E-06" ixz="2E-06" iyy="0.004831" iyz="0.000448" izz="0.001409" />
-      </inertial>
-      <visual>
-        <origin xyz="0 0 0" rpy="0 0 0" />
-        <geometry>
-          <mesh filename="file://$(find robot_description)/meshes/shoulder_link.STL" />
-        </geometry>
-        <material name="">
-          <color rgba="0.75294 0.75294 0.75294 1" />
-        </material>
-      </visual>
-      <collision>
-        <origin xyz="0 0 0" rpy="0 0 0" />
-        <geometry>
-          <mesh filename="file://$(find robot_description)/meshes/shoulder_link.STL" />
-        </geometry>
-      </collision>
-    </link>
-    <joint name="${prefix}joint_1" type="continuous">
-      <origin xyz="0 0 0.15643" rpy="-3.1416 0.0 0.0" />
-      <parent link="${prefix}base_link" />
-      <child link="${prefix}shoulder_link" />
-      <axis xyz="0 0 1" />
-      <limit effort="39" velocity="1.3963" />
-    </joint>
-    <link name="${prefix}bicep_link">
-      <inertial>
-        <origin xyz="3.5E-05 -0.208207 -0.01889" rpy="0 0 0" />
-        <mass value="1.262" />
-        <inertia ixx="0.046752" ixy="-9E-06" ixz="0" iyy="0.00085" iyz="-9.8E-05" izz="0.047188" />
-      </inertial>
-      <visual>
-        <origin xyz="0 0 0" rpy="0 0 0" />
-        <geometry>
-          <mesh filename="file://$(find robot_description)/meshes/bicep_link.STL" />
-        </geometry>
-        <material name="">
-          <color rgba="0.75294 0.75294 0.75294 1" />
-        </material>
-      </visual>
-      <collision>
-        <origin xyz="0 0 0" rpy="0 0 0" />
-        <geometry>
-          <mesh filename="file://$(find robot_description)/meshes/bicep_link.STL" />
-        </geometry>
-      </collision>
-    </link>
-    <joint name="${prefix}joint_2" type="revolute">
-      <origin xyz="0 0.005375 -0.12838" rpy="1.5708 0.0 0.0" />
-      <parent link="${prefix}shoulder_link" />
-      <child link="${prefix}bicep_link" />
-      <axis xyz="0 0 1" />
-      <limit lower="-2.24" upper="2.24" effort="39" velocity="1.3963" />
-    </joint>
-    <link name="${prefix}forearm_link">
-      <inertial>
-        <origin xyz="1.8E-05 0.076168 -0.01397" rpy="0 0 0" />
-        <mass value="0.93" />
-        <inertia ixx="0.008292" ixy="-1E-06" ixz="0" iyy="0.000628" iyz="0.000432" izz="0.008464" />
-      </inertial>
-      <visual>
-        <origin xyz="0 0 0" rpy="0 0 0" />
-        <geometry>
-          <mesh filename="file://$(find robot_description)/meshes/forearm_link.STL" />
-        </geometry>
-        <material name="">
-          <color rgba="0.75294 0.75294 0.75294 1" />
-        </material>
-      </visual>
-      <collision>
-        <origin xyz="0 0 0" rpy="0 0 0" />
-        <geometry>
-          <mesh filename="file://$(find robot_description)/meshes/forearm_link.STL" />
-        </geometry>
-      </collision>
-    </link>
-    <joint name="${prefix}joint_3" type="revolute">
-      <origin xyz="0 -0.41 0" rpy="3.1416 0 0" />
-      <parent link="${prefix}bicep_link" />
-      <child link="${prefix}forearm_link" />
-      <axis xyz="0 0 1" />
-      <limit lower="-2.57" upper="2.57" effort="39" velocity="1.3963" />
-    </joint>
-    <link name="${prefix}spherical_wrist_1_link">
-      <inertial>
-        <origin xyz="-1E-06 0.008486 -0.062937" rpy="0 0 0" />
-        <mass value="0.6781" />
-        <inertia ixx="0.001645" ixy="0" ixz="0" iyy="0.001666" iyz="-0.000234" izz="0.000389" />
-      </inertial>
-      <visual>
-        <origin xyz="0 0 0" rpy="0 0 0" />
-        <geometry>
-          <mesh filename="file://$(find robot_description)/meshes/spherical_wrist_1_link.STL" />
-        </geometry>
-        <material name="">
-          <color rgba="0.75294 0.75294 0.75294 1" />
-        </material>
-      </visual>
-      <collision>
-        <origin xyz="0 0 0" rpy="0 0 0" />
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
Commit message: [New] ros2_controllers. Joint position controller.

File: src/robot_description/urdf/gen3_macro.xacro (robot description, xacro)
@@ -261,4 +261,82 @@
         <child  link="${prefix}camera_color_frame" />
       </joint>
+  <!-- Control -->
+       <ros2_control name="GazeboSystem" type="system">
+          <hardware>
+            <plugin>gazebo_ros2_control/GazeboSystem</plugin>
+          </hardware>
+          <joint name="joint_1">
+            <command_interface name="position">
+              <param name="min">-1000</param>
+              <param name="max">1000</param>
+            </command_interface>
+            <state_interface name="position">
+              <param name="initial_value">1.0</param>
+            </state_interface>
+            <state_interface name="velocity"/>
+            <state_interface name="effort"/>
+          </joint>
+             <joint name="joint_2">
+            <command_interface name="position">
+              <param name="min">-1000</param>
+              <param name="max">1000</param>
+            </command_interface>
+            <state_interface name="position">
+              <param name="initial_value">1.0</param>
+            </state_interface>
+            <state_interface name="velocity"/>
+            <state_interface name="effort"/>
+          </joint>
+             <joint name="joint_3">
+            <command_interface name="position">
+              <param name="min">-1000</param>
+              <param name="max">1000</param>
+            </command_interface>
+            <state_interface name="position">
+              <param name="initial_value">1.0</param>
+            </state_interface>
+            <state_interface name="velocity"/>
+            <state_interface name="effort"/>
+          </joint>
+             <joint name="joint_4">
+            <command_interface name="position">
+              <param name="min">-1000</param>
+              <param name="max">1000</param>
+            </command_interface>
+            <state_interface name="position">
+              <param name="initial_value">1.0</param>
+            </state_interface>
+            <state_interface name="velocity"/>
+            <state_interface name="effort"/>
+          </joint>
+             <joint name="joint_5">
+            <command_interface name="position">
+              <param name="min">-1000</param>
+              <param name="max">1000</param>
+            </command_interface>
+            <state_interface name="position">
+              <param name="initial_value">1.0</param>
+            </state_interface>
+            <state_interface name="velocity"/>
+            <state_interface name="effort"/>
+          </joint>
+             <joint name="joint_6">
+            <command_interface name="position">
+              <param name="min">-1000</param>
+              <param name="max">1000</param>
+            </command_interface>
+            <state_interface name="position">
+              <param name="initial_value">1.0</param>
+            </state_interface>
+            <state_interface name="velocity"/>
+            <state_interface name="effort"/>
+          </joint>
+        </ros2_control>
+<gazebo>
+   <plugin filename="libgazebo_ros2_control.so" name="gazebo_ros2_control">
+      <parameters>$(find robot_description)/config/robot_controller.yaml</parameters>
+    </plugin>
+</gazebo>
+  <!-- gazebo -->
    <gazebo reference="${prefix}camera_link">
     <sensor type="depth" name="intel_camera">
