Commit message: [New] functional trajectory movement in gazebo

File: src/robot_description/urdf/gen3_macro.xacro (robot description, xacro)
@@ -58,5 +58,5 @@
       <child link="${prefix}shoulder_link" />
       <axis xyz="0 0 1" />
-      <limit effort="39" velocity="1.3963" />
+      <limit effort="39" velocity="40" />
     </joint>
     <link name="${prefix}bicep_link">
@@ -87,5 +87,5 @@
       <child link="${prefix}bicep_link" />
       <axis xyz="0 0 1" />
-      <limit lower="-2.24" upper="2.24" effort="39" velocity="1.3963" />
+      <limit lower="-2.24" upper="2.24" effort="39" velocity="40" />
     </joint>
     <link name="${prefix}forearm_link">
@@ -116,5 +116,5 @@
       <child link="${prefix}forearm_link" />
       <axis xyz="0 0 1" />
-      <limit lower="-2.57" upper="2.57" effort="39" velocity="1.3963" />
+      <limit lower="-2.57" upper="2.57" effort="39" velocity="40" />
     </joint>
     <link name="${prefix}spherical_wrist_1_link">
@@ -145,5 +145,5 @@
       <child link="${prefix}spherical_wrist_1_link" />
       <axis xyz="0 0 1" />
-      <limit effort="9" velocity="1.2218" />
+      <limit effort="9" velocity="40" />
     </joint>
     <link name="${prefix}spherical_wrist_2_link">
@@ -174,5 +174,5 @@
       <child link="${prefix}spherical_wrist_2_link" />
       <axis xyz="0 0 1" />
-      <limit lower="-2.09" upper="2.09" effort="9" velocity="1.2218" />
+      <limit lower="-2.09" upper="2.09" effort="9" velocity="40" />
     </joint>
     <xacro:if value="${vision}">
@@ -229,5 +229,5 @@
       <child link="${prefix}bracelet_link" />
       <axis xyz="0 0 1" />
-      <limit effort="9" velocity="1.2218" />
+      <limit effort="9" velocity="40" />
     </joint>
     <link name="${prefix}end_effector_link" />
@@ -272,8 +272,7 @@
             </command_interface>
             <state_interface name="position">
-              <param name="initial_value">1.0</param>
-            </state_interface>
-            <state_interface name="velocity"/>
-            <state_interface name="effort"/>
+              <!-- <param name="initial_value">0.0</param> -->
+            </state_interface>
+            <state_interface name="velocity"/>
           </joint>
              <joint name="joint_2">
@@ -283,8 +282,7 @@
             </command_interface>
             <state_interface name="position">
-              <param name="initial_value">1.0</param>
-            </state_interface>
-            <state_interface name="velocity"/>
-            <state_interface name="effort"/>
+              <!-- <param name="initial_value">1.0</param> -->
+            </state_interface>
+            <state_interface name="velocity"/>
           </joint>
              <joint name="joint_3">
@@ -294,8 +292,7 @@
             </command_interface>
             <state_interface name="position">
-              <param name="initial_value">1.0</param>
-            </state_interface>
-            <state_interface name="velocity"/>
-            <state_interface name="effort"/>
+              <!-- <param name="initial_value">1.0</param> -->
+            </state_interface>
+            <state_interface name="velocity"/>
           </joint>
              <joint name="joint_4">
@@ -305,8 +302,7 @@
             </command_interface>
             <state_interface name="position">
-              <param name="initial_value">1.0</param>
-            </state_interface>
-            <state_interface name="velocity"/>
-            <state_interface name="effort"/>
+              <!-- <param name="initial_value">1.0</param> -->
+            </state_interface>
+            <state_interface name="velocity"/>
           </joint>
              <joint name="joint_5">
@@ -316,8 +312,7 @@
             </command_interface>
             <state_interface name="position">
-              <param name="initial_value">1.0</param>
-            </state_interface>
-            <state_interface name="velocity"/>
-            <state_interface name="effort"/>
+              <!-- <param name="initial_value">1.0</param> -->
+            </state_interface>
+            <state_interface name="velocity"/>
           </joint>
              <joint name="joint_6">
@@ -327,8 +322,7 @@
             </command_interface>
             <state_interface name="position">
-              <param name="initial_value">1.0</param>
-            </state_interface>
-            <state_interface name="velocity"/>
-            <state_interface name="effort"/>
+              <!-- <param name="initial_value">1.0</param> -->
+            </state_interface>
+            <state_interface name="velocity"/>
           </joint>
         </ros2_control>

Commit message: [Update] Camera final

File: src/robot_description/urdf/gen3_macro.xacro (robot description, xacro)
@@ -245,5 +245,5 @@
       <link name="${prefix}camera_link" />
       <joint name="${prefix}camera_module" type="fixed">
-        <origin xyz="0.2 0.05639 -0.00305" rpy="3.14159265358979 3.14159265358979 0" />
+        <origin xyz="0 0.05639 -0.00305" rpy="3.14159265358979 3.14159265358979 0" />
         <parent link="${prefix}end_effector_link" />
         <child  link="${prefix}camera_link" />
@@ -355,6 +355,6 @@
           <alwaysOn>true</alwaysOn>
               <updateRate>10.0</updateRate>
-              <cameraName>your_camera</cameraName>
-              <frameName>your_camera_link</frameName>
+              <cameraName>inter_camera</cameraName>
+              <frameName>camera_link</frameName>
           <imageTopicName>rgb/image_raw</imageTopicName>
           <depthImageTopicName>depth/image_raw</depthImageTopicName>
