Commit message: [Update] Gripper added

File: src/robot_description/grippers/gen3_lite_2f/urdf/gen3_lite_2f_macro.xacro (robot description, xacro)
@@ -26,5 +26,5 @@
         <origin xyz="0 0 0" rpy="0 0 0" />
         <geometry>
-          <mesh filename="package://kortex_description/grippers/gen3_lite_2f/meshes/gripper_base_link.STL" />
+          <mesh filename="file://$(find robot_description)/grippers/gen3_lite_2f/meshes/gripper_base_link.STL" />
         </geometry>
         <material name="">
@@ -35,5 +35,5 @@
         <origin xyz="0 0 0" rpy="0 0 0" />
         <geometry>
-          <mesh filename="package://kortex_description/grippers/gen3_lite_2f/meshes/gripper_base_link.STL" />
+          <mesh filename="file://$(find robot_description)/grippers/gen3_lite_2f/meshes/gripper_base_link.STL" />
         </geometry>
       </collision>
@@ -51,5 +51,5 @@
       <origin xyz="0 0 0" rpy="0 0 0" />
       <geometry>
-        <mesh filename="package://kortex_description/grippers/gen3_lite_2f/meshes/right_finger_prox_link.STL" />
+        <mesh filename="file://$(find robot_description)/grippers/gen3_lite_2f/meshes/right_finger_prox_link.STL" />
       </geometry>
       <material name="">
@@ -60,5 +60,5 @@
       <origin xyz="0 0 0" rpy="0 0 0" />
       <geometry>
-        <mesh filename="package://kortex_description/grippers/gen3_lite_2f/meshes/right_finger_prox_link.STL" />
+        <mesh filename="file://$(find robot_description)/grippers/gen3_lite_2f/meshes/right_finger_prox_link.STL" />
       </geometry>
     </collision>
@@ -83,5 +83,5 @@
         <origin xyz="0 0 0" rpy="0 0 0" />
         <geometry>
-          <mesh filename="package://kortex_description/grippers/gen3_lite_2f/meshes/right_finger_dist_link.STL" />
+          <mesh filename="file://$(find robot_description)/grippers/gen3_lite_2f/meshes/right_finger_dist_link.STL" />
         </geometry>
         <material name="">
@@ -92,5 +92,5 @@
         <origin xyz="0 0 0" rpy="0 0 0" />
         <geometry>
-          <mesh filename="package://kortex_description/grippers/gen3_lite_2f/meshes/right_finger_dist_link.STL" />
+          <mesh filename="file://$(find robot_description)/grippers/gen3_lite_2f/meshes/right_finger_dist_link.STL" />
         </geometry>
       </collision>
@@ -116,5 +116,5 @@
         <origin xyz="0 0 0" rpy="0 0 0" />
         <geometry>
-          <mesh filename="package://kortex_description/grippers/gen3_lite_2f/meshes/left_finger_prox_link.STL" />
+          <mesh filename="file://$(find robot_description)/grippers/gen3_lite_2f/meshes/left_finger_prox_link.STL" />
         </geometry>
         <material name="">
@@ -125,5 +125,5 @@
         <origin xyz="0 0 0" rpy="0 0 0" />
         <geometry>
-          <mesh filename="package://kortex_description/grippers/gen3_lite_2f/meshes/left_finger_prox_link.STL" />
+          <mesh filename="file://$(find robot_description)/grippers/gen3_lite_2f/meshes/left_finger_prox_link.STL" />
         </geometry>
       </collision>
@@ -149,5 +149,5 @@
         <origin xyz="0 0 0" rpy="0 0 0" />
         <geometry>
-          <mesh filename="package://kortex_description/grippers/gen3_lite_2f/meshes/left_finger_dist_link.STL" />
+          <mesh filename="file://$(find robot_description)/grippers/gen3_lite_2f/meshes/left_finger_dist_link.STL" />
         </geometry>
         <material name="">
@@ -158,5 +158,5 @@
         <origin xyz="0 0 0" rpy="0 0 0" />
         <geometry>
-          <mesh filename="package://kortex_description/grippers/gen3_lite_2f/meshes/left_finger_dist_link.STL" />
+          <mesh filename="file://$(find robot_description)/grippers/gen3_lite_2f/meshes/left_finger_dist_link.STL" />
         </geometry>
       </collision>

File: src/robot_description/grippers/robotiq_2f_140/urdf/robotiq_arg2f.xacro (robot description, xacro)
@@ -18,6 +18,6 @@
         <geometry>
           <!-- The DAE file doesn't show well in Gazebo so we're using the STL instead -->
-          <!-- <mesh filename="package://kortex_description/grippers/robotiq_2f_140/meshes/visual/robotiq_arg2f_140_base_link.dae" scale="0.001 0.001 0.001"/> -->
-          <mesh filename="package://kortex_description/grippers/robotiq_2f_140/meshes/collision/robotiq_arg2f_base_link.stl" />
+          <!-- <mesh filename="file://$(find robot_description)/grippers/robotiq_2f_140/meshes/visual/robotiq_arg2f_140_base_link.dae" scale="0.001 0.001 0.001"/> -->
+          <mesh filename="file://$(find robot_description)/grippers/robotiq_2f_140/meshes/collision/robotiq_arg2f_base_link.stl" />
         </geometry>
         <material name="">
@@ -28,5 +28,5 @@
         <origin xyz="0 0 0" rpy="0 0 0" />
         <geometry>
-          <mesh filename="package://kortex_description/grippers/robotiq_2f_140/meshes/collision/robotiq_arg2f_base_link.stl" />
+          <mesh filename="file://$(find robot_description)/grippers/robotiq_2f_140/meshes/collision/robotiq_arg2f_base_link.stl" />
         </geometry>
       </collision>

File: src/robot_description/grippers/robotiq_2f_140/urdf/robotiq_arg2f_140_model_macro.xacro (robot description, xacro)
@@ -17,5 +17,5 @@
         <origin xyz="0 0 0" rpy="0 0 0" />
         <geometry>
-          <mesh filename="package://kortex_description/grippers/robotiq_2f_140/meshes/visual/robotiq_arg2f_${stroke}_outer_knuckle.stl" />
+          <mesh filename="file://$(find robot_description)/grippers/robotiq_2f_140/meshes/visual/robotiq_arg2f_${stroke}_outer_knuckle.stl" />
         </geometry>
         <material name="">
@@ -26,5 +26,5 @@
         <origin xyz="0 0 0" rpy="0 0 0" />
         <geometry>
-          <mesh filename="package://kortex_description/grippers/robotiq_2f_140/meshes/collision/robotiq_arg2f_${stroke}_outer_knuckle.stl" />
+          <mesh filename="file://$(find robot_description)/grippers/robotiq_2f_140/meshes/collision/robotiq_arg2f_${stroke}_outer_knuckle.stl" />
         </geometry>
       </collision>
@@ -55,5 +55,5 @@
         <origin xyz="0 0 0" rpy="0 0 0" />
         <geometry>
-          <mesh filename="package://kortex_description/grippers/robotiq_2f_140/meshes/visual/robotiq_arg2f_${stroke}_outer_finger.stl" />
+          <mesh filename="file://$(find robot_description)/grippers/robotiq_2f_140/meshes/visual/robotiq_arg2f_${stroke}_outer_finger.stl" />
         </geometry>
         <material name="">
@@ -64,5 +64,5 @@
         <origin xyz="0 0 0" rpy="0 0 0" />
         <geometry>
-          <mesh filename="package://kortex_description/grippers/robotiq_2f_140/meshes/collision/robotiq_arg2f_${stroke}_outer_finger.stl" />
+          <mesh filename="file://$(find robot_description)/grippers/robotiq_2f_140/meshes/collision/robotiq_arg2f_${stroke}_outer_finger.stl" />
         </geometry>
       </collision>
@@ -88,5 +88,5 @@
         <origin xyz="0 0 0" rpy="0 0 0" />
         <geometry>
-          <mesh filename="package://kortex_description/grippers/robotiq_2f_140/meshes/visual/robotiq_arg2f_${stroke}_inner_knuckle.stl" />
+          <mesh filename="file://$(find robot_description)/grippers/robotiq_2f_140/meshes/visual/robotiq_arg2f_${stroke}_inner_knuckle.stl" />
         </geometry>
         <material name="">
@@ -97,5 +97,5 @@
         <origin xyz="0 0 0" rpy="0 0 0" />
         <geometry>
-          <mesh filename="package://kortex_description/grippers/robotiq_2f_140/meshes/collision/robotiq_arg2f_${stroke}_inner_knuckle.stl" />
+          <mesh filename="file://$(find robot_description)/grippers/robotiq_2f_140/meshes/collision/robotiq_arg2f_${stroke}_inner_knuckle.stl" />
         </geometry>
       </collision>
@@ -121,5 +121,5 @@
         <origin xyz="0 0 0" rpy="0 0 0" />
         <geometry>
-          <mesh filename="package://kortex_description/grippers/robotiq_2f_140/meshes/visual/robotiq_arg2f_${stroke}_inner_finger.stl" />
+          <mesh filename="file://$(find robot_description)/grippers/robotiq_2f_140/meshes/visual/robotiq_arg2f_${stroke}_inner_finger.stl" />
         </geometry>
         <material name="">
@@ -130,5 +130,5 @@
         <origin xyz="0 0 0" rpy="0 0 0" />
         <geometry>
-          <mesh filename="package://kortex_description/grippers/robotiq_2f_140/meshes/collision/robotiq_arg2f_${stroke}_inner_finger.stl" />
+          <mesh filename="file://$(find robot_description)/grippers/robotiq_2f_140/meshes/collision/robotiq_arg2f_${stroke}_inner_finger.stl" />
         </geometry>
       </collision>

File: src/robot_description/grippers/robotiq_2f_85/urdf/robotiq_2f_85_macro.xacro (robot description, xacro)
@@ -2,5 +2,5 @@
 <robot name="robotiq_arg2f_85_model" xmlns:xacro="http://ros.org/wiki/xacro">
   <xacro:macro name="load_gripper" params="parent prefix">
-    <xacro:include filename="$(find kortex_description)/grippers/robotiq_2f_85/urdf/robotiq_arg2f_85_model_macro.xacro" />
+    <xacro:include filename="$(find robot_description)/grippers/robotiq_2f_85/urdf/robotiq_arg2f_85_model_macro.xacro" />
     <xacro:robotiq_arg2f_85 parent="${parent}" prefix="${prefix}"/>
   </xacro:macro>

File: src/robot_description/grippers/robotiq_2f_85/urdf/robotiq_arg2f.xacro (robot description, xacro)
@@ -18,6 +18,6 @@
         <geometry>
           <!-- The DAE file doesn't show well in Gazebo so we're using the STL instead -->
-          <!-- <mesh filename="package://kortex_description/grippers/robotiq_2f_85/meshes/visual/robotiq_arg2f_85_base_link.dae" scale="0.001 0.001 0.001"/> -->
-          <mesh filename="package://kortex_description/grippers/robotiq_2f_85/meshes/collision/robotiq_arg2f_base_link.stl" />
+          <!-- <mesh filename="file://$(find robot_description)/grippers/robotiq_2f_85/meshes/visual/robotiq_arg2f_85_base_link.dae" scale="0.001 0.001 0.001"/> -->
+          <mesh filename="file://$(find robot_description)/grippers/robotiq_2f_85/meshes/collision/robotiq_arg2f_base_link.stl" />
         </geometry>
         <material name="">
@@ -28,5 +28,5 @@
         <origin xyz="0 0 0" rpy="0 0 0" />
         <geometry>
-           <mesh filename="package://kortex_description/grippers/robotiq_2f_85/meshes/collision/robotiq_arg2f_base_link.stl" />
+           <mesh filename="file://$(find robot_description)/grippers/robotiq_2f_85/meshes/collision/robotiq_arg2f_base_link.stl" />
         </geometry>
       </collision>

File: src/robot_description/grippers/robotiq_2f_85/urdf/robotiq_arg2f_85_model_macro.xacro (robot description, xacro)
@@ -13,5 +13,5 @@
         <origin xyz="0 0 0" rpy="0 0 0" />
         <geometry>
-          <mesh filename="package://kortex_description/grippers/robotiq_2f_85/meshes/visual/robotiq_arg2f_85_outer_knuckle.dae" scale="0.001 0.001 0.001"/>
+          <mesh filename="file://$(find robot_description)/grippers/robotiq_2f_85/meshes/visual/robotiq_arg2f_85_outer_knuckle.dae" scale="0.001 0.001 0.001"/>
         </geometry>
         <material name="">
@@ -22,5 +22,5 @@
         <origin xyz="0 0 0" rpy="0 0 0" />
         <geometry>
-          <mesh filename="package://kortex_description/grippers/robotiq_2f_85/meshes/collision/robotiq_arg2f_85_outer_knuckle.dae" scale="0.001 0.001 0.001"/>
+          <mesh filename="file://$(find robot_description)/grippers/robotiq_2f_85/meshes/collision/robotiq_arg2f_85_outer_knuckle.dae" scale="0.001 0.001 0.001"/>
         </geometry>
       </collision>
@@ -37,5 +37,5 @@
         <origin xyz="0 0 0" rpy="0 0 0" />
         <geometry>
-          <mesh filename="package://kortex_description/grippers/robotiq_2f_85/meshes/visual/robotiq_arg2f_85_outer_finger.dae" scale="0.001 0.001 0.001"/>
+          <mesh filename="file://$(find robot_description)/grippers/robotiq_2f_85/meshes/visual/robotiq_arg2f_85_outer_finger.dae" scale="0.001 0.001 0.001"/>
         </geometry>
         <material name="">
@@ -46,5 +46,5 @@
         <origin xyz="0 0 0" rpy="0 0 0" />
         <geometry>
-          <mesh filename="package://kortex_description/grippers/robotiq_2f_85/meshes/collision/robotiq_arg2f_85_outer_finger.dae" scale="0.001 0.001 0.001"/>
+          <mesh filename="file://$(find robot_description)/grippers/robotiq_2f_85/meshes/collision/robotiq_arg2f_85_outer_finger.dae" scale="0.001 0.001 0.001"/>
         </geometry>
       </collision>
@@ -61,5 +61,5 @@
         <origin xyz="0 0 0" rpy="0 0 0" />
         <geometry>
-          <mesh filename="package://kortex_description/grippers/robotiq_2f_85/meshes/visual/robotiq_arg2f_85_inner_knuckle.dae" scale="0.001 0.001 0.001"/>
+          <mesh filename="file://$(find robot_description)/grippers/robotiq_2f_85/meshes/visual/robotiq_arg2f_85_inner_knuckle.dae" scale="0.001 0.001 0.001"/>
         </geometry>
         <material name="">
@@ -70,5 +70,5 @@
         <origin xyz="0 0 0" rpy="0 0 0" />
         <geometry>
-          <mesh filename="package://kortex_description/grippers/robotiq_2f_85/meshes/collision/robotiq_arg2f_85_inner_knuckle.dae" scale="0.001 0.001 0.001"/>
+          <mesh filename="file://$(find robot_description)/grippers/robotiq_2f_85/meshes/collision/robotiq_arg2f_85_inner_knuckle.dae" scale="0.001 0.001 0.001"/>
         </geometry>
       </collision>
@@ -85,5 +85,5 @@
         <origin xyz="0 0 0" rpy="0 0 0" />
         <geometry>
-          <mesh filename="package://kortex_description/grippers/robotiq_2f_85/meshes/visual/robotiq_arg2f_85_inner_finger.dae" scale="0.001 0.001 0.001"/>
+          <mesh filename="file://$(find robot_description)/grippers/robotiq_2f_85/meshes/visual/robotiq_arg2f_85_inner_finger.dae" scale="0.001 0.001 0.001"/>
         </geometry>
         <material name="">
@@ -94,5 +94,5 @@
         <origin xyz="0 0 0" rpy="0 0 0" />
         <geometry>
-          <mesh filename="package://kortex_description/grippers/robotiq_2f_85/meshes/collision/robotiq_arg2f_85_inner_finger.dae" scale="0.001 0.001 0.001" />
+          <mesh filename="file://$(find robot_description)/grippers/robotiq_2f_85/meshes/collision/robotiq_arg2f_85_inner_finger.dae" scale="0.001 0.001 0.001" />
         </geometry>
       </collision>
@@ -159,5 +159,5 @@
     </joint>
   </xacro:macro>
-  <xacro:include filename="$(find kortex_description)/grippers/robotiq_2f_85/urdf/robotiq_arg2f.xacro" />
+  <xacro:include filename="$(find robot_description)/grippers/robotiq_2f_85/urdf/robotiq_arg2f.xacro" />
   <xacro:macro name="finger_joint" params="prefix">
     <joint name="${prefix}finger_joint" type="revolute">

File: src/robot_description/urdf/GEN3-6DOF_BRAKES_NO-VISION_URDF_ARM_V01.urdf (robot description, URDF)
Before this commit: robot GEN3-6DOF_BRAKES_NO-VISION_URDF_ARM_V01, 8 links, 7 joints
Links:
- link base_link: geometry collision mesh filename=file://$(find robot_description)/arms/gen3/6dof/meshes/base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; visual mesh filename=file://$(find robot_description)/arms/gen3/6dof/meshes/base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
- link bicep_link: geometry collision mesh filename=file://$(find robot_description)/arms/gen3/6dof/meshes/bice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; visual mesh filename=file://$(find robot_description)/arms/gen3/6dof/meshes/bice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
- link bracelet_link: geometry collision mesh filename=file://$(find robot_description)/arms/gen3/6dof/meshes/brac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; visual mesh filename=file://$(find robot_description)/arms/gen3/6dof/meshes/brac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
- link forearm_link: geometry collision mesh filename=file://$(find robot_description)/arms/gen3/6dof/meshes/fore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; visual mesh filename=file://$(find robot_description)/arms/gen3/6dof/meshes/fore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
- link shoulder_link: geometry collision mesh filename=file://$(find robot_description)/arms/gen3/6dof/meshes/shou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; visual mesh filename=file://$(find robot_description)/arms/gen3/6dof/meshes/shou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
- link spherical_wrist_1_link: geometry collision mesh filename=file://$(find robot_description)/arms/gen3/6dof/meshes/sphe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; visual mesh filename=file://$(find robot_description)/arms/gen3/6dof/meshes/sphe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
- link spherical_wrist_2_link: geometry collision mesh filename=file://$(find robot_description)/arms/gen3/6dof/meshes/sphe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; visual mesh filename=file://$(find robot_description)/arms/gen3/6dof/meshes/sphe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

File: src/robot_description/urdf/GEN3-6DOF_BRAKES_VISION_URDF_ARM_V01.urdf (robot description, URDF)
Before this commit: robot GEN3-6DOF_BRAKES_VISION_URDF_ARM_V01, 11 links, 10 joints
Links:
- link base_link: geometry collision mesh filename=file://$(find robot_description)/arms/gen3/6dof/meshes/base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; visual mesh filename=file://$(find robot_description)/arms/gen3/6dof/meshes/base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
- link bicep_link: geometry collision mesh filename=file://$(find robot_description)/arms/gen3/6dof/meshes/bice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; visual mesh filename=file://$(find robot_description)/arms/gen3/6dof/meshes/bice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
- link bracelet_link: geometry collision mesh filename=file://$(find robot_description)/arms/gen3/6dof/meshes/brac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; visual mesh filename=file://$(find robot_description)/arms/gen3/6dof/meshes/brac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
- link forearm_link: geometry collision mesh filename=file://$(find robot_description)/arms/gen3/6dof/meshes/fore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; visual mesh filename=file://$(find robot_description)/arms/gen3/6dof/meshes/fore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
- link shoulder_link: geometry collision mesh filename=file://$(find robot_description)/arms/gen3/6dof/meshes/shou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; visual mesh filename=file://$(find robot_description)/arms/gen3/6dof/meshes/shou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
- link spherical_wrist_1_link: geometry collision mesh filename=file://$(find robot_description)/arms/gen3/6dof/meshes/sphe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; visual mesh filename=file://$(find robot_description)/arms/gen3/6dof/meshes/sphe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
- link spherical_wrist_2_link: geometry collision mesh filename=file://$(find robot_description)/arms/gen3/6dof/meshes/sphe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; visual mesh filename=file://$(find robot_description)/arms/gen3/6dof/meshes/sphe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

File: src/robot_description/urdf/GEN3-6DOF_NO-VISION_URDF_ARM_V01.urdf (robot description, URDF)
Before this commit: robot GEN3-6DOF_NO-VISION_URDF_ARM_V01, 8 links, 7 joints
Links:
- link base_link: geometry collision mesh filename=file://$(find robot_description)/arms/gen3/6dof/meshes/base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; visual mesh filename=file://$(find robot_description)/arms/gen3/6dof/meshes/base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
- link bicep_link: geometry collision mesh filename=file://$(find robot_description)/arms/gen3/6dof/meshes/bice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; visual mesh filename=file://$(find robot_description)/arms/gen3/6dof/meshes/bice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
- link bracelet_link: geometry collision mesh filename=file://$(find robot_description)/arms/gen3/6dof/meshes/brac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; visual mesh filename=file://$(find robot_description)/arms/gen3/6dof/meshes/brac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
- link forearm_link: geometry collision mesh filename=file://$(find robot_description)/arms/gen3/6dof/meshes/fore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; visual mesh filename=file://$(find robot_description)/arms/gen3/6dof/meshes/fore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
- link shoulder_link: geometry collision mesh filename=file://$(find robot_description)/arms/gen3/6dof/meshes/shou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; visual mesh filename=file://$(find robot_description)/arms/gen3/6dof/meshes/shou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
- link spherical_wrist_1_link: geometry collision mesh filename=file://$(find robot_description)/arms/gen3/6dof/meshes/sphe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; visual mesh filename=file://$(find robot_description)/arms/gen3/6dof/meshes/sphe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
- link spherical_wrist_2_link: geometry collision mesh filename=file://$(find robot_description)/arms/gen3/6dof/meshes/sphe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; visual mesh filename=file://$(find robot_description)/arms/gen3/6dof/meshes/sphe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

File: src/robot_description/urdf/GEN3-6DOF_VISION_URDF_ARM_V01.urdf (robot description, URDF)
Before this commit: robot GEN3-6DOF_VISION_URDF_ARM_V01, 11 links, 10 joints
Links:
- link base_link: geometry collision mesh filename=file://$(find robot_description)/arms/gen3/6dof/meshes/base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; visual mesh filename=file://$(find robot_description)/arms/gen3/6dof/meshes/base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
- link bicep_link: geometry collision mesh filename=file://$(find robot_description)/arms/gen3/6dof/meshes/bice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; visual mesh filename=file://$(find robot_description)/arms/gen3/6dof/meshes/bice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
- link bracelet_link: geometry collision mesh filename=file://$(find robot_description)/arms/gen3/6dof/meshes/brac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; visual mesh filename=file://$(find robot_description)/arms/gen3/6dof/meshes/brac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
- link forearm_link: geometry collision mesh filename=file://$(find robot_description)/arms/gen3/6dof/meshes/fore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; visual mesh filename=file://$(find robot_description)/arms/gen3/6dof/meshes/fore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
- link shoulder_link: geometry collision mesh filename=file://$(find robot_description)/arms/gen3/6dof/meshes/shou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; visual mesh filename=file://$(find robot_description)/arms/gen3/6dof/meshes/shou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
- link spherical_wrist_1_link: geometry collision mesh filename=file://$(find robot_description)/arms/gen3/6dof/meshes/sphe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; visual mesh filename=file://$(find robot_description)/arms/gen3/6dof/meshes/sphe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
- link spherical_wrist_2_link: geometry collision mesh filename=file://$(find robot_description)/arms/gen3/6dof/meshes/sphe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; visual mesh filename=file://$(find robot_description)/arms/gen3/6dof/meshes/sphe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

File: src/robot_description/urdf/gen3_macro.xacro (robot description, xacro)
@@ -4,9 +4,14 @@
   <xacro:property name="last_arm_link" value="end_effector_link"/>
   <xacro:macro name="load_arm" params="parent:='' dof vision prefix *origin">
-  <link name="world" />
+  <!-- <link name="world" />
   <joint name="world_to_base_link=" type="fixed">
      <parent link="world"/>
      <child link="base_link"/>
-  </joint>
+  </joint> -->
+  <!-- Gripper  -->
+  <!-- <joint name ="ee_joint" type="fixed">
+       <parent link="end_effector_link"/>
+       <child link="robotiq_2f_85"/>
+  </joint> -->
     <link name="${prefix}base_link">
       <inertial>

File: src/robot_description/xacro/gen3.xacro (robot description, xacro)
@@ -3,5 +3,5 @@
     <!-- Arguments -->
     <xacro:arg name="arm" default="gen3" />
-    <xacro:arg name="dof" default="7" />
+    <xacro:arg name="dof" default="6" />
     <xacro:arg name="vision" default="true" />
     <xacro:arg name="gripper" default="" />
